File: KiCAD/hv-signal-gen/hv-signal-gen.kicad_sch (KiCad schematic)
At the start: 17 parts, among them J1 Conn_01x05, SW1 SW_SPST_GND

Commit message: initial software
Parts:
- removed C2: .01uF 250V, symbol Device:C
- removed C3: 100uF 250V, symbol Device:C_Polarized
- removed C4: 22uF 250V, symbol Device:C_Polarized
- added A1: Arduino_Nano_v3.x, Module:Arduino_Nano, symbol MCU_Module:Arduino_Nano_v3.x
- added R13, R15, R16: 100k, symbol Device:R_US
- added R14: 100R 2W, symbol Device:R_US
- C5, C6: value 22uF 250V -> 22uF 100V
- D2, D3: value 70V zener -> 66V 2W Zener
- R2: value 100R 2W -> 1k
- R3: value 1k -> 100k
- R4: value 4.7k -> 1k
Connections:
- net +5V: now also A1.27 (+5V)
- net GND: now also R3.1, A1.29 (GND), A1.4 (GND), R15.2
- net HV_DAC1/FUNC_OUT: now also R16.1
- net HV_DAC2/FUNC_OUT: now also R13.1
- net -65V: now reaches R2.2
- net -65V: now also C6.2, D3.2 (A), R15.1; no longer R3.1
- net at R4.1: now also C1.1, R1.2; no longer R3.2
- net +75V renamed +65V
- net +65V: now also R3.2
- removed net -75V: C1.2, C6.2, D1.3 (-), D3.2 (A)
- new net: C1.2, R14.2, R2.1
- new net: D1.3 (-), R14.1
- new net CS0: A1.11 (D8)
- new net CS1: A1.12 (D9)
- new net MISO: A1.15 (D12)
- new net MOSI: A1.14 (D11)
- new net SCK: A1.16 (D13)
- new net SCL: A1.24 (A5)
- new net SDA: A1.23 (A4)
- new net SS: A1.13 (D10)
- new net ~{LDAC}: A1.10 (D7)
Other:
- note added: "+/-65V regulated supply"
- note added: "HV OUT!"
- note removed: "+/-70V regulated supply"
- moved on the sheet: C5, C6, D2, D3, R4
