File: KiCAD/hv-signal-gen/hv_dac.kicad_sch (KiCad schematic)
At the start: 12 parts, among them U1 MCP4921, U2 LTC6090

Commit message: initial software
Parts:
- removed R5: 40kΩ, Resistor_SMD:R_1206_3216Metric_Pad1.30x1.75mm_HandSolder, symbol Device:R_US
Connections:
- net HV_OA is gone; now on net FUNC_OUT: C11.2, R8.2, U2.6
Changed lines of the file:
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@@
 	(wire
 		(pts
-			(xy 184.15 97.79) (xy 193.04 97.79)
+			(xy 184.15 97.79) (xy 214.63 97.79)
 		)
 		(stroke
@@
 		(pts
 			(xy 87.63 101.6) (xy 106.68 101.6)
-		)
-		(stroke
-			(width 0)
-			(type default)
-		)
-	)
-	(wire
-		(pts
-			(xy 200.66 97.79) (xy 214.63 97.79)
 		)
 		(stroke
@@
 					(unit 1)
 				)
-			)
-		)
-	)
-	(symbol
-		(lib_id "Device:R_US")
-		(at 196.85 97.79 90)
-		(unit 1)
-		(exclude_from_sim no)
-		(in_bom yes)
-		(on_board yes)
-		(dnp no)
-		(property "Reference" "R5"
-			(at 196.85 92.71 90)
-			(effects
-				(font
-					(size 1.27 1.27)
-				)
-			)
-		)
-		(property "Value" "40kΩ"
-			(at 196.85 95.25 90)
-			(effects
-				(font
-					(size 1.27 1.27)
-				)
-			)
-		)
-		(property "Footprint" "Resistor_SMD:R_1206_3216Metric_Pad1.30x1.75mm_HandSolder"
-			(at 197.104 96.774 90)
-			(effects
-				(font
-					(size 1.27 1.27)
-				)
-				(hide yes)
-			)
-		)
-		(property "Datasheet" "~"
-			(at 196.85 97.79 0)
-			(effects
-				(font
-					(size 1.27 1.27)
-				)
-				(hide yes)
-			)
-		)
-		(property "Description" ""
-			(at 196.85 97.79 0)
-			(effects
-				(font
-					(size 1.27 1.27)
-				)
-			)
-		)
-		(pin "1"
-		)
-		(pin "2"
-		)
-		(instances
-			(project "hv-signal-gen"
-				(path "/bd3461c6-98d5-44ba-aae5-a7d4c774348f/2a705cc3-c219-4e7d-8713-06178cfed8dd"
-					(reference "R13")
-					(unit 1)
-				)
-				(path "/bd3461c6-98d5-44ba-aae5-a7d4c774348f/c6ed43be-e184-41ee-ae2b-489664e00d43"
-					(reference "R5")
-					(unit 1)
-				)
