File: KiCAD/Arduino_Shield_V2_Erics/PCB.kicad_sch (KiCad schematic)
At the start: 20 parts, among them J1 Power, J2 Digital/PWM, J3 Analog, J4 Digital/PWM, J5 Conn_01x01, J6 Conn_01x01_Socket, J7 Conn_01x01, J8 Conn_01x01, U1 MCP4921, U2 LTC6090

Commit message: Update documentation
Connections:
- net 8 is gone; now on net *6: J2.10 (Pin_10)
Other:
- note added: "For 2nd channel, cut or bend out long pin on J4 pin 2 (U1 pin 2 connection) Add wire from J4 pin 2 to J2 pin 8"
- note added: "Green wire on board#2 only"
- note removed: "For 2nd channel, cut long pin on J4 pin 2 (U1 pin 2 connection) Add wire from J4 pin 2 to J2 pin 8"
Changed lines of the file:
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@@
 		)
 	)
-	(text "For 2nd channel, cut long pin\non J4 pin 2 (U1 pin 2 connection)\n\nAdd wire from J4 pin 2 to J2 pin 8"
+	(text "For 2nd channel, cut or bend out long pin\non J4 pin 2 (U1 pin 2 connection)\n\nAdd wire from J4 pin 2 to J2 pin 8"
 		(exclude_from_sim no)
-		(at 59.69 126.492 0)
+		(at 55.372 128.524 0)
 		(effects
 			(font
@@
 			)
 			(justify left bottom)
+		)
+	)
+	(text "Green wire on\nboard#2 only"
+		(exclude_from_sim no)
+		(at 70.612 90.932 0)
+		(effects
+			(font
+				(size 1.27 1.27)
+			)
+			(justify left)
 		)
 	)
@@
 	)
 	(junction
+		(at 85.09 100.33)
+		(diameter 0)
+		(color 0 0 0 0)
+	)
+	(junction
 		(at 166.37 71.12)
 		(diameter 0)
@@
 	(wire
 		(pts
-			(xy 67.31 100.33) (xy 95.25 100.33)
+			(xy 67.31 100.33) (xy 85.09 100.33)
 		)
 		(stroke
@@
 	(wire
 		(pts
+			(xy 80.01 87.63) (xy 85.09 87.63)
+		)
+		(stroke
+			(width 0.635)
+			(type default)
+			(color 0 255 0 1)
+		)
+	)
+	(wire
+		(pts
 			(xy 118.11 71.12) (xy 110.49 71.12)
 		)
@@
 	(wire
 		(pts
+			(xy 85.09 87.63) (xy 85.09 100.33)
+		)
+		(stroke
+			(width 0.635)
+			(type default)
+			(color 0 255 0 1)
+		)
+	)
+	(wire
+		(pts
 			(xy 67.31 64.77) (xy 80.01 64.77)
 		)
@@
 	(wire
 		(pts
-			(xy 69.85 72.39) (xy 69.85 90.17)
+			(xy 68.58 72.39) (xy 68.58 90.17)
 		)
 		(stroke
@@
 	(wire
 		(pts
-			(xy 67.31 72.39) (xy 69.85 72.39)
+			(xy 67.31 72.39) (xy 68.58 72.39)
 		)
 		(stroke
@@
 			(type solid)
 			(color 0 0 255 1)
+		)
+	)
+	(wire
+		(pts
+			(xy 85.09 100.33) (xy 95.25 100.33)
+		)
+		(stroke
+			(width 0)
+			(type default)
 		)
 	)
@@
 	(symbol
 		(lib_id "power:GND")
-		(at 69.85 90.17 0)
+		(at 68.58 90.17 0)
 		(unit 1)
 		(exclude_from_sim no)
@@
 		(dnp no)
 		(property "Reference" "#PWR05"
-			(at 69.85 96.52 0)
+			(at 68.58 96.52 0)
 			(effects
 				(font
@@
 		)
 		(property "Value" "GND"
-			(at 69.85 93.98 0)
+			(at 68.58 93.98 0)
 			(effects
 				(font
@@
 		)
 		(property "Footprint" ""
-			(at 69.85 90.17 0)
+			(at 68.58 90.17 0)
 			(effects
 				(font
@@
 		)
 		(property "Datasheet" ""
-			(at 69.85 90.17 0)
+			(at 68.58 90.17 0)
 			(effects
 				(font
@@
 		)
 		(property "Description" ""
-			(at 69.85 90.17 0)
-			(effects
-				(font
+			(at 68.58 90.17 0)
+			(effects
+				(font
